File: output/pcbs/pcb.kicad_pcb (KiCad board)
At the start: 2 copper layers, 158.2 x 134.4 mm, 68 parts

Commit message: wired pcb
Parts:
- moved D28 4.00 mm to (256.0, 177.3), turned to 70 degrees
- moved D29 4.00 mm to (262.5, 159.3), turned to 70 degrees
- moved D1 4.00 mm to (146.0, 155.0), turned to 90 degrees
- moved D10 4.00 mm to (184.0, 126.0), turned to 90 degrees
- moved D11 4.00 mm to (184.0, 107.0), turned to 90 degrees
- moved D12 4.00 mm to (184.0, 88.0), turned to 90 degrees
- moved D13 4.00 mm to (203.0, 140.0), turned to 90 degrees
- moved D14 4.00 mm to (203.0, 121.0), turned to 90 degrees
- moved D15 4.00 mm to (203.0, 102.0), turned to 90 degrees
- moved D16 4.00 mm to (203.0, 83.0), turned to 90 degrees
- moved D17 4.00 mm to (222.0, 145.0), turned to 90 degrees
- moved D18 4.00 mm to (222.0, 126.0), turned to 90 degrees
- moved D19 4.00 mm to (222.0, 107.0), turned to 90 degrees
- moved D2 4.00 mm to (146.0, 136.0), turned to 90 degrees
- moved D20 4.00 mm to (222.0, 88.0), turned to 90 degrees
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